File: Hardware/Logics WIP/FLD Logic (autorouted).sch (EAGLE design)
At the start: 86 parts

Commit message: 
Parts:
- removed H1, H2, H3, H4: MOUNT-HOLE3.3, holes:MOUNT-HOLE3.3
Changed lines of the file:
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@@
 <part name="GND81" library="supply0" deviceset="GND" device=""/>
 <part name="OUT" library="pinhead" deviceset="PINHD-1X3" device=""/>
-<part name="H1" library="holes" deviceset="MOUNT-HOLE" device="3.3"/>
-<part name="H2" library="holes" deviceset="MOUNT-HOLE" device="3.3"/>
-<part name="H3" library="holes" deviceset="MOUNT-HOLE" device="3.3"/>
-<part name="H4" library="holes" deviceset="MOUNT-HOLE" device="3.3"/>
 <part name="V9" library="supply0" deviceset="+5V" device=""/>
 <part name="GND3" library="supply0" deviceset="GND" device=""/>
@@
 <instance part="GND81" gate="1" x="297.18" y="-73.66"/>
 <instance part="OUT" gate="A" x="325.12" y="213.36"/>
-<instance part="H1" gate="G$1" x="-7.62" y="-81.28"/>
-<instance part="H2" gate="G$1" x="0" y="170.18"/>
-<instance part="H3" gate="G$1" x="391.16" y="160.02"/>
-<instance part="H4" gate="G$1" x="381" y="-76.2"/>
 <instance part="V9" gate="1" x="266.7" y="213.36" rot="R90"/>
 <instance part="GND3" gate="1" x="274.32" y="226.06" rot="R180"/>
